File: Hardware/Nixie-Controller-v2.sch (KiCad schematic (older format))
At the start: 209 parts

Commit message: Assign footprint to test points
Parts:
- TP? (x5): footprint (none) -> TestPoint:TestPoint_Pad_D2.5mm
- TP? (x9): footprint (none) -> TestPoint:TestPoint_Pad_D1.5mm
Changed lines of the file:
@@
 F 0 "TP?" V 28400 2588 50  0000 L CNN
 F 1 "~" H 28458 2427 50  0000 L CNN
-F 2 "" H 28600 2400 50  0001 C CNN
+F 2 "TestPoint:TestPoint_Pad_D1.5mm" H 28600 2400 50  0001 C CNN
 F 3 "~" H 28600 2400 50  0001 C CNN
 F 4 "~" H 28400 2400 50  0001 C CNN "Manufacturer"
@@
 F 0 "TP?" V 28400 2738 50  0000 L CNN
 F 1 "~" H 28458 2577 50  0000 L CNN
-F 2 "" H 28600 2550 50  0001 C CNN
+F 2 "TestPoint:TestPoint_Pad_D1.5mm" H 28600 2550 50  0001 C CNN
 F 3 "~" H 28600 2550 50  0001 C CNN
 F 4 "~" H 28400 2550 50  0001 C CNN "Manufacturer"
@@
 F 0 "TP?" V 28400 2888 50  0000 L CNN
 F 1 "~" H 28458 2727 50  0000 L CNN
-F 2 "" H 28600 2700 50  0001 C CNN
+F 2 "TestPoint:TestPoint_Pad_D1.5mm" H 28600 2700 50  0001 C CNN
 F 3 "~" H 28600 2700 50  0001 C CNN
 F 4 "~" H 28400 2700 50  0001 C CNN "Manufacturer"
@@
 F 0 "TP?" V 28400 3188 50  0000 L CNN
 F 1 "~" H 28458 3027 50  0000 L CNN
-F 2 "" H 28600 3000 50  0001 C CNN
+F 2 "TestPoint:TestPoint_Pad_D1.5mm" H 28600 3000 50  0001 C CNN
 F 3 "~" H 28600 3000 50  0001 C CNN
 F 4 "~" H 28400 3000 50  0001 C CNN "Manufacturer"
@@
 F 0 "TP?" V 29200 2588 50  0000 L CNN
 F 1 "~" H 29258 2427 50  0000 L CNN
-F 2 "" H 29400 2400 50  0001 C CNN
+F 2 "TestPoint:TestPoint_Pad_D1.5mm" H 29400 2400 50  0001 C CNN
 F 3 "~" H 29400 2400 50  0001 C CNN
 F 4 "~" H 29200 2400 50  0001 C CNN "Manufacturer"
@@
 F 0 "TP?" V 29200 2738 50  0000 L CNN
 F 1 "~" H 29258 2577 50  0000 L CNN
-F 2 "" H 29400 2550 50  0001 C CNN
+F 2 "TestPoint:TestPoint_Pad_D1.5mm" H 29400 2550 50  0001 C CNN
 F 3 "~" H 29400 2550 50  0001 C CNN
 F 4 "~" H 29200 2550 50  0001 C CNN "Manufacturer"
@@
 F 0 "TP?" V 29200 2888 50  0000 L CNN
 F 1 "~" H 29258 2727 50  0000 L CNN
-F 2 "" H 29400 2700 50  0001 C CNN
+F 2 "TestPoint:TestPoint_Pad_D1.5mm" H 29400 2700 50  0001 C CNN
 F 3 "~" H 29400 2700 50  0001 C CNN
 F 4 "~" H 29200 2700 50  0001 C CNN "Manufacturer"
@@
 F 0 "TP?" V 29200 3038 50  0000 L CNN
 F 1 "~" H 29258 2877 50  0000 L CNN
-F 2 "" H 29400 2850 50  0001 C CNN
+F 2 "TestPoint:TestPoint_Pad_D1.5mm" H 29400 2850 50  0001 C CNN
 F 3 "~" H 29400 2850 50  0001 C CNN
 F 4 "~" H 29200 2850 50  0001 C CNN "Manufacturer"
@@
 F 0 "TP?" V 29200 3188 50  0000 L CNN
 F 1 "~" H 29258 3027 50  0000 L CNN
-F 2 "" H 29400 3000 50  0001 C CNN
+F 2 "TestPoint:TestPoint_Pad_D1.5mm" H 29400 3000 50  0001 C CNN
 F 3 "~" H 29400 3000 50  0001 C CNN
 F 4 "~" H 29200 3000 50  0001 C CNN "Manufacturer"
@@
 F 0 "TP?" V 30950 2450 50  0000 L CNN
 F 1 "3.3V" V 31050 2450 50  0000 L CNN
-F 2 "" H 31200 2250 50  0001 C CNN
+F 2 "TestPoint:TestPoint_Pad_D2.5mm" H 31200 2250 50  0001 C CNN
 F 3 "~" H 31200 2250 50  0001 C CNN
+F 4 "~" H 31000 2250 50  0001 C CNN "Manufacturer"
+F 5 "~" H 31000 2250 50  0001 C CNN "Part#"
 	1    31000 2250
 	0    1    1    0
@@
 F 0 "TP?" V 30950 2700 50  0000 L CNN
 F 1 "5V" V 31050 2700 50  0000 L CNN
-F 2 "" H 31200 2500 50  0001 C CNN
+F 2 "TestPoint:TestPoint_Pad_D2.5mm" H 31200 2500 50  0001 C CNN
 F 3 "~" H 31200 2500 50  0001 C CNN
+F 4 "~" H 31000 2500 50  0001 C CNN "Manufacturer"
+F 5 "~" H 31000 2500 50  0001 C CNN "Part#"
 	1    31000 2500
 	0    1    1    0
@@
 F 0 "TP?" V 30950 2950 50  0000 L CNN
 F 1 "12V" V 31050 2950 50  0000 L CNN
-F 2 "" H 31200 2750 50  0001 C CNN
+F 2 "TestPoint:TestPoint_Pad_D2.5mm" H 31200 2750 50  0001 C CNN
 F 3 "~" H 31200 2750 50  0001 C CNN
+F 4 "~" H 31000 2750 50  0001 C CNN "Manufacturer"
+F 5 "~" H 31000 2750 50  0001 C CNN "Part#"
 	1    31000 2750
 	0    1    1    0
@@
 F 0 "TP?" V 30950 3200 50  0000 L CNN
 F 1 "180V" V 31050 3200 50  0000 L CNN
-F 2 "" H 31200 3000 50  0001 C CNN
+F 2 "TestPoint:TestPoint_Pad_D2.5mm" H 31200 3000 50  0001 C CNN
 F 3 "~" H 31200 3000 50  0001 C CNN
+F 4 "~" H 31000 3000 50  0001 C CNN "Manufacturer"
+F 5 "~" H 31000 3000 50  0001 C CNN "Part#"
 	1    31000 3000
 	0    1    1    0
@@
 F 0 "TP?" V 30950 3450 50  0000 L CNN
 F 1 "GND" V 31050 3450 50  0000 L CNN
-F 2 "" H 31200 3250 50  0001 C CNN
+F 2 "TestPoint:TestPoint_Pad_D2.5mm" H 31200 3250 50  0001 C CNN
 F 3 "~" H 31200 3250 50  0001 C CNN
+F 4 "~" H 31000 3250 50  0001 C CNN "Manufacturer"
+F 5 "~" H 31000 3250 50  0001 C CNN "Part#"
 	1    31000 3250
 	0    1    1    0

Commit message: Add RTC
Parts:
- added BT?: BACKUP, Battery:BatteryHolder_Keystone_1058_1x2032, symbol Device:Battery_Cell
- added C?: 100nF, Capacitor_SMD:C_0402_1005Metric, symbol Device:C_Small
- added R? (x3): 6.8K, Resistor_SMD:R_0402_1005Metric, symbol Device:R_Small_US
- added TP?: BATT, TestPoint:TestPoint_Pad_D2.5mm, symbol Connector:TestPoint
- added TP?: RTC_CAL, TestPoint:TestPoint_Pad_D2.5mm, symbol Connector:TestPoint
- added U?: M41T01, Package_SO:SOIC-8_3.9x4.9mm_P1.27mm, symbol Nixie-Controller-v2:M41T01
- added Y?: 32.768KHz, Crystal:Crystal_SMD_2012-2Pin_2.0x1.2mm, symbol Device:Crystal_Small
Connections:
- net +3V3: now also C?.1, R?.1, R?.1, R?.1, U?.8 (VCC)
- net GND: now also BT?.2 (-), C?.2, U?.4 (VSS)
- new net: U?.1 (OSC1), Y?.1
- new net: U?.2 (OSC2), Y?.2
- new net: R?.2, TP?.1, U?.7 (TEST)
- new net +BATT: BT?.1 (+), TP?.1, U?.3 (VBAT)
- new net RTC_SCL: R?.2, U?.6 (SCL)
- new net RTC_SDA: R?.2, U?.5 (SDA)
Other:
- note added: "REAL TIME CLOCK"
- moved on the sheet: TP?

Commit message: Fix DRC issues
Parts:
- gave numbers to parts that had none: 218
Connections:
- net RTC_SCL: now also U20.42 (PB6)
- net RTC_SDA: now also U20.43 (PB7)
- no-connect marks 45 -> 66

Commit message: Add DC barrel jack
Parts:
- added J7: 12V DC JACK, Connector_BarrelJack:BarrelJack_Horizontal, symbol Connector:Conn_01x02_Female
- renumbered C5 to C10, C12 to C11, C19 to C12, C6 to C13, C13 to C14, C25 to C15, C26 to C16, C27 to C17, C28 to C18, C29 to C19, C3 to C2, C30 to C20, C33 to C21, C7 to C22, C14 to C23, C31 to C24, C32 to C25, C8 to C26, C15 to C27, C9 to C28, C16 to C29, C20 to C3, C10 to C30, C17 to C31, C11 to C32, C18 to C33, C21 to C4, C22 to C5, C23 to C6, C24 to C7, C4 to C8, C2 to C9, Q50 to Q10, Q56 to Q11, Q3 to Q12, Q9 to Q13, Q15 to Q14, Q21 to Q15, Q27 to Q16, Q33 to Q17, Q39 to Q18, Q45 to Q19, Q51 to Q20, Q57 to Q21, Q4 to Q22, Q10 to Q23, Q16 to Q24, Q22 to Q25, Q28 to Q26, Q34 to Q27, Q40 to Q28, Q46 to Q29, Q8 to Q3, Q52 to Q30, Q58 to Q31, Q5 to Q32, Q11 to Q33, Q17 to Q34, Q23 to Q35, Q29 to Q36, Q35 to Q37, Q41 to Q38, Q47 to Q39, Q14 to Q4, Q53 to Q40, Q59 to Q41, Q6 to Q42, Q12 to Q43, Q18 to Q44, Q24 to Q45, Q30 to Q46, Q36 to Q47, Q42 to Q48, Q48 to Q49, Q20 to Q5, Q54 to Q50, Q60 to Q51, Q7 to Q52, Q13 to Q53, Q19 to Q54, Q25 to Q55, Q31 to Q56, Q37 to Q57, Q43 to Q58, Q49 to Q59, Q26 to Q6, Q55 to Q60, Q32 to Q7, Q38 to Q8, Q44 to Q9, R2 to R1, R46 to R10, R52 to R11, R58 to R12, R64 to R13, R34 to R14, R71 to R15, R72 to R16, R73 to R17, R5 to R18, R11 to R19, R1 to R2, R17 to R20, R23 to R21, R29 to R22, R41 to R23, R47 to R24, R53 to R25, R59 to R26, R65 to R27, R70 to R28, R35 to R29, R6 to R30, R12 to R31, R18 to R32, R24 to R33, R30 to R34, R42 to R35, R48 to R36, R54 to R37, R60 to R38, R66 to R39, R36 to R40, R7 to R41, R13 to R42, R19 to R43, R25 to R44, R31 to R45, R43 to R46, R49 to R47, R55 to R48, R61 to R49, R10 to R5, R67 to R50, R37 to R51, R8 to R52, R14 to R53, R20 to R54, R26 to R55, R32 to R56, R44 to R57, R50 to R58, R56 to R59, R16 to R6, R62 to R60, R68 to R61, R38 to R62, R9 to R63, R15 to R64, R21 to R65, R27 to R66, R33 to R67, R45 to R68, R51 to R69, R22 to R7, R57 to R70, R63 to R71, R69 to R72, R39 to R73, R28 to R8, R40 to R9, TP11 to TP1, TP9 to TP10, TP14 to TP11, TP5 to TP12, TP10 to TP13, TP15 to TP14, TP16 to TP15, TP1 to TP16, TP12 to TP2, TP2 to TP3, TP6 to TP4, TP3 to TP5, TP7 to TP6, TP13 to TP7, TP4 to TP8, TP8 to TP9, U8 to U1, U9 to U10, U22 to U11, U20 to U12, U2 to U13, U10 to U14, U3 to U15, U11 to U16, U4 to U17, U12 to U18, U5 to U19, U16 to U2, U13 to U20, U6 to U21, U14 to U22, U17 to U3, U18 to U4, U19 to U5, U21 to U6, U15 to U8, U1 to U9, Y2 to Y1, Y1 to Y2
Connections:
- net +12V: now also J7.1 (Pin_1)
- net GND: now also J7.2 (Pin_2)
