File: Nixie-Controller-v2.kicad_pcb (KiCad board)
At the start: 4 copper layers, 220 x 65 mm, 228 parts, among them J7 12V DC JACK, J8 RST, U1 MAX1771, U10 74HC4067, U11 M41T01, U12 STM32F103C8, U13 OPA180, U14 74HC4067, U15 OPA180, U16 74HC4067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

Commit message: Migrate to KiCAD 6
Other:
- net class Default removed
